File: Hardware/EuroSID.kicad_pcb (KiCad board)
At the start: 2 copper layers, 213.3 x 106.6 mm, 232 parts, among them J1 GATE_2, J10 IN_2, J11 IN_3, J12 PWM_CV, J13 EXT_CON, J14 Conn_01x04_Female, J15 Eurorack Connector, J16 Conn_01x06_Male, J17 Conn_ARM_JTAG_SWD_10, J18 Power_Connector_IO, J19 Power_Connector, J2 GATE_3, J20 Digital_Connector_IO, J21 CV_Connector_IO, J22 Pot_Connector_IO, J23 Attenuverter_Connector_IO, J24 Digital_Connector, J25 CV_Connector, J26 Pot_Connector, J27 Attenuverter_Connector, J28 SID_Audio_Connector_IO, J29 SID_Audio_Connector, J3 GATE_1, J4 OUT2_CON, J5 CUTOFF_CV, J6 SHAPE_CV, J7 SET_CV, J8 OUT1_CON, J9 IN_1, Q1 MMBT3904, Q2 MMBT3904, Q3 MMBT3904, SW1 Frequency Adjust, SW10 SET_SW, SW11 FILTER_SW, SW12 FILTEREXT_SW, SW13 SHAPE_SW, SW2 MOD_SW, SW3 FILTER1_SW, SW4 PROG, SW5 VOICE_SW, SW6 FILTER2_SW, SW7 RST, SW8 MODE_SW, SW9 FILTER3_SW, U1 TLC5947DAP, U10 LM1117-3.3, U11 LM1117-5.0, U12 L7809, U13 STM32F303RBTx, U2 OPA1678, U3 MCP6004, U4 MCP6004, U6 74HC595, U7 74HC595, U8 SID, U9 LM1117-3.3, X1 ECS-8FMX-010-TR

Commit message: Moved SID chip to backside
Parts:
- J14, JP1, U8: moved to B.Cu
- J15: footprint Connector_PinHeader_2.54mm:PinHeader_2x08_P2.54mm_Vertical -> Connector_IDC:IDC-Header_2x08_P2.54mm_Vertical; moved to B.Cu
- J19: moved to F.Cu
- J25, J26: footprint Connector_PinSocket_2.54mm:PinSocket_2x04_P2.54mm_Vertical -> Connector_PinHeader_2.54mm:PinHeader_2x04_P2.54mm_Vertical
- J27: footprint Connector_PinSocket_2.54mm:PinSocket_1x04_P2.54mm_Vertical -> Connector_PinHeader_2.54mm:PinHeader_1x04_P2.54mm_Vertical
- RV5, RV6, RV7, RV8: footprint Potentiometer_THT:Potentiometer_Bourns_PTA2043_Single_Slide -> Potentiometer_THT:Potentiometer_Bourns_PTL20_Single_Slide
- moved J20 166.7 mm to (327.5, -14.5)
- moved J21 166.7 mm to (345.7, -21.3)
- moved J22 166.7 mm to (361.5, -5.08)
- moved J23 166.7 mm to (349.3, -4.83)
- moved J28 166.7 mm to (313.6, -1.53)
- moved U1 166.7 mm to (362.6, -24.5)
- moved J18 166.7 mm to (312.9, -19.6)
- moved RV7 130.0 mm to (174.0, 55.1)
- moved RV5 108.9 mm to (160.3, 55.1)
- moved C3 96.1 mm to (273.3, 20.6)
- moved RV6 94.0 mm to (187.2, 55.1)
- moved RV8 92.0 mm to (200.5, 55.1)
- moved J29 86.4 mm to (47.5, 55.6)
- moved J25 81.9 mm to (131.9, 47.5)
- moved J24 80.9 mm to (135.4, 80.0)
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Routing:
- net +5V: track 146.1 -> 93.7 mm
- net /SID Chip/D0: track 8.90 -> 40.2 mm
- net /SID Chip/D1: track 7.63 -> 38.3 mm, vias 0 -> 2
- net Net-(D26-Pad1): track 6.61 -> 36.5 mm
- net /SID Chip/A3: track 29.1 -> 6.26 mm
- net /SID Chip/A2: track 32.3 -> 10.7 mm
- net /SID Chip/A1: track 35.6 -> 15.1 mm
- net /SID Chip/A0: track 39.2 -> 19.3 mm
- net /SID Chip/D2: track 6.90 -> 23.2 mm, vias 0 -> 2
- net /SID Chip/D3: track 6.37 -> 22.4 mm, vias 0 -> 2
- net /SID Chip/A4: track 28.4 -> 12.6 mm, vias 2 -> 1
- net /SID Chip/D4: track 5.85 -> 21.6 mm, vias 0 -> 2
- net /SID Chip/D5: track 5.32 -> 21.0 mm, vias 0 -> 2
- net /SID Chip/D6: track 5.76 -> 21.4 mm
- net /SID Chip/D7: track 12.7 -> 27.4 mm
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- removed copper zone on B.Cu, net GND
